Commit message: Added kinect sensor

File: frobo_description/urdf/frobo.urdf (robot description, URDF)
Before this commit: robot Frobo, 4 links, 3 joints
Links:
- added link head_camera_frame; collision box size=0.064 0.28 0.04; visual mesh filename=package://frobo_description/meshes/kinect.stl
- added link head_camera_ir_link; visual sphere radius=0.0005
- added link head_camera_ir_optical_frame
- added link head_camera_rgb_link; visual sphere radius=0.0005
- added link head_camera_rgb_optical_frame
Joints:
- added joint head_camera_frame_joint: type fixed, parent base_link, child head_camera_frame, origin xyz=0 0 0.26 rpy=0 0 0
- added joint head_camera_ir_joint: type fixed, parent head_camera_frame, child head_camera_ir_link, origin xyz=0 0 0 rpy=0 0 0
- added joint head_camera_ir_optical_frame_joint: type fixed, parent head_camera_ir_link, child head_camera_ir_optical_frame, origin xyz=0 0 0 rpy=-1.57 0.0 -1.57
- added joint head_camera_rgb_joint: type fixed, parent head_camera_ir_link, child head_camera_rgb_link, origin xyz=0 -0.03 0 rpy=0 0 0
- added joint head_camera_rgb_optical_frame_joint: type fixed, parent head_camera_rgb_link, child head_camera_rgb_optical_frame, origin xyz=0 0 0 rpy=-1.57 0.0 -1.57

File: frobo_description/urdf/frobo.urdf.xacro (robot description, xacro)
@@ -4,5 +4,10 @@
   <include filename="$(find frobo_description)/urdf/base.urdf.xacro" />
   <include filename="$(find frobo_description)/urdf/materials.urdf.xacro" />
+  <include filename="$(find frobo_description)/urdf/kinect_camera.urdf.xacro" />
   <!-- Now we can start using the macros included above to define the actual Frobo -->
   <frobo_base name="base" color="Brown"/>
+  <!-- Camera -->
+  <kinect_camera name="head_camera" parent="base_link">
+    <origin xyz="0 0 0.26" rpy="0 0 0"/>
+  </kinect_camera>
 </robot>
