Commit message: frobo_description: updating kinect position

File: frobo_description/urdf/frobo.urdf.xacro (robot description, xacro)
@@ -14,5 +14,5 @@
   <!-- Camera -->
   <kinect_camera name="head_camera" parent="base_link">
-    <origin xyz="0 0.002 0.345" rpy="0 0 0"/>
+    <origin xyz="-0.015 0.002 0.345" rpy="0 0 0"/>
   </kinect_camera>
   <!-- Lidar -->
