Commit message: frobo_description: updated URDF model with lidar and layers

File: frobo_description/urdf/base.urdf.xacro (robot description, xacro)
@@ -2,4 +2,7 @@
 <robot>
   <property name="ground_clearance" value="0.0740" />
+  <property name="level1_clearance" value="0.18" />
+  <property name="level2_clearance" value="0.24" />
+  <property name="level3_clearance" value="0.305" />
   <property name="wheel_offset_y" value="0.116" />
   <property name="wheel_length" value="0.02032" />
@@ -60,4 +63,25 @@
         <material name="${color}" />
       </visual>
+      <visual>
+        <origin xyz="0 0 ${level1_clearance}" rpy="0 0 0" />
+        <geometry>
+	  <cylinder radius="${base_radius}" length="${base_length}"/>
+        </geometry>
+        <material name="${color}" />
+      </visual>
+      <visual>
+        <origin xyz="0 0 ${level2_clearance}" rpy="0 0 0" />
+        <geometry>
+	  <cylinder radius="${base_radius}" length="${base_length}"/>
+        </geometry>
+        <material name="${color}" />
+      </visual>
+      <visual>
+        <origin xyz="0 0 ${level3_clearance}" rpy="0 0 0" />
+        <geometry>
+	  <cylinder radius="${base_radius}" length="${base_length}"/>
+        </geometry>
+        <material name="${color}" />
+      </visual>
       <!-- fixed wheels, without tf transform, just for visualization -->
       <visual>

File: frobo_description/urdf/frobo.urdf (robot description, URDF)
Before this commit: robot Frobo, 9 links, 8 joints
Links:
- added link lidar_link; visual cylinder length=0.05211 radius=0.05
- link base_link: geometry collision cylinder length=0.12382 radius=0.2; visual cylinder length=0.006 radius=0.15
Joints:
- added joint lidar_joint: type fixed, parent base_link, child lidar_link, origin xyz=-0.02 0 0.285 rpy=0 0 0
- joint head_camera_frame_joint: origin xyz=0 0 0.26 rpy=0 0 0 -> xyz=0 0 0.35 rpy=0 0 0

File: frobo_description/urdf/frobo.urdf.xacro (robot description, xacro)
@@ -5,9 +5,14 @@
   <include filename="$(find frobo_description)/urdf/materials.urdf.xacro" />
   <include filename="$(find frobo_description)/urdf/kinect_camera.urdf.xacro" />
+  <include filename="$(find frobo_description)/urdf/lidar.urdf.xacro" />
   <!-- Now we can start using the macros included above to define the actual Frobo -->
   <frobo_base name="base" color="Brown"/>
   <!-- Camera -->
   <kinect_camera name="head_camera" parent="base_link">
-    <origin xyz="0 0 0.26" rpy="0 0 0"/>
+    <origin xyz="0 0 0.35" rpy="0 0 0"/>
   </kinect_camera>
+  <!-- Lidar -->
+  <lidar name="lidar" parent="base_link">
+    <origin xyz="-0.02 0 0.285" rpy="0 0 0"/>
+  </lidar>
 </robot>

Commit message: First gazebo version

File: frobo_description/urdf/base.urdf.xacro (robot description, xacro)
@@ -1,20 +1,21 @@
 <?xml version="1.0"?>
-<robot>
-  <property name="ground_clearance" value="0.0740" />
-  <property name="level1_clearance" value="0.18" />
-  <property name="level2_clearance" value="0.24" />
-  <property name="level3_clearance" value="0.305" />
-  <property name="wheel_offset_y" value="0.116" />
-  <property name="wheel_length" value="0.02032" />
-  <property name="wheel_radius" value="0.06191" />
-  <property name="swivel_length" value="0.019" />
-  <property name="swivel_radius" value="0.025" />
-  <property name="base_radius" value="0.15" />
-  <property name="base_collision_radius" value="0.20" />
-  <property name="base_length" value="0.006" />
-  <property name="sonar_clearance" value="${ground_clearance-0.02}" />
-  <property name="sonar_angle" value="0.6" />
+<robot xmlns:xacro="http://www.ros.org/wiki/xacro">
+  <xacro:property name="ground_clearance" value="0.0740" />
+  <xacro:property name="level1_clearance" value="0.18" />
+  <xacro:property name="level2_clearance" value="0.24" />
+  <xacro:property name="level3_clearance" value="0.305" />
+  <xacro:property name="wheel_offset_y" value="0.116" />
+  <xacro:property name="wheel_length" value="0.02032" />
+  <xacro:property name="wheel_radius" value="0.06191" />
+  <xacro:property name="swivel_length" value="0.019" />
+  <xacro:property name="swivel_radius" value="0.025" />
+  <xacro:property name="base_radius" value="0.15" />
+  <xacro:property name="base_collision_radius" value="0.20" />
+  <xacro:property name="base_collision_top_clearance" value="0.10" />
+  <xacro:property name="base_length" value="0.006" />
+  <xacro:property name="sonar_clearance" value="${ground_clearance-0.02}" />
+  <xacro:property name="sonar_angle" value="0.6" />
   <!-- define a rotating wheel -->
-  <macro name="frobo_wheel" params="suffix parent reflect color">
+  <xacro:macro name="frobo_wheel" params="suffix parent reflect color">
     <joint name="${parent}_${suffix}_wheel_joint" type="continuous">
       <axis xyz="0 0 1" />
@@ -33,8 +34,22 @@
         <material name="${color}" />
       </visual>
+      <collision>
+        <origin xyz="0 0 0" rpy="0 0 0" />
+        <geometry>
+          <cylinder radius="${wheel_radius}" length="${wheel_length}"/>
+        </geometry>
+      </collision>
+      <inertial>
+        <origin xyz="0 0 ${wheel_radius}" rpy="0 0 0"/>
+        <mass value="0.2"/>
+        <inertia
+          ixx="1e-3" ixy="0.0" ixz="0.0"
+          iyy="1e-3" iyz="0.0"
+          izz="1e-3"/>
+      </inertial>
     </link>
-  </macro>
+  </xacro:macro>
   <!-- define a sonar -->
-  <macro name="frobo_sonar" params="suffix parent offset_x offset_y angle color">
+  <xacro:macro name="frobo_sonar" params="suffix parent offset_x offset_y angle color">
     <joint name="${parent}_${suffix}_sonar_joint" type="fixed">
       <origin xyz="${offset_x} ${offset_y} ${sonar_clearance}" rpy="0 0 ${angle}" />
@@ -51,7 +66,7 @@
       </visual>
     </link>
-  </macro>
+  </xacro:macro>
   <!-- The xacro macro frobo_base contains: base and wheels -->
-  <macro name="frobo_base" params="name color">
+  <xacro:macro name="frobo_base" params="name color">
     <link name="${name}_link">
       <visual>
@@ -110,9 +125,17 @@
       -->
       <collision>
-        <origin xyz="0 0 ${wheel_radius}" rpy="0 0 0" />
+        <origin xyz="0 0 ${(level3_clearance+base_collision_top_clearance)/2}" rpy="0 0 0" />
         <geometry>
-          <cylinder radius="${base_collision_radius}" length="${wheel_radius*2}" />
+          <cylinder radius="${base_collision_radius}" length="${level3_clearance+base_collision_top_clearance}"/>
         </geometry>
       </collision>
+      <inertial>
+        <origin xyz="0 0 ${base_radius}" rpy="0 0 0"/>
+        <mass value="5"/>
+        <inertia
+          ixx="10e-3" ixy="0.0" ixz="0.0"
+          iyy="10e-3" iyz="0.0"
+          izz="10e-3"/>
+      </inertial>
     </link>
     <!-- drive wheels -->
@@ -123,4 +146,4 @@
     <frobo_sonar parent="${name}" offset_x="0.125" offset_y="0" angle="0" suffix="fc" color="Blue"/>
     <frobo_sonar parent="${name}" offset_x="0.115" offset_y="0.055" angle="${sonar_angle}" suffix="fl" color="Blue"/>
-  </macro>
+  </xacro:macro>
 </robot>

File: frobo_description/urdf/frobo.urdf (robot description, URDF)
Before this commit: robot Frobo, 10 links, 9 joints
Links:
- link base_link: mass None -> 5; geometry collision cylinder length=0.405 radius=0.2; visual cylinder length=0.006 radius=0.15

File: frobo_description/urdf/frobo.urdf.xacro (robot description, xacro)
@@ -1,9 +1,12 @@
 <?xml version="1.0"?>
-<robot name="Frobo" >
+<robot name="frobo" xmlns:xacro="http://www.ros.org/wiki/xacro">
   <!-- The following included files set up definitions of parts of the robot body -->
-  <include filename="$(find frobo_description)/urdf/base.urdf.xacro" />
-  <include filename="$(find frobo_description)/urdf/materials.urdf.xacro" />
-  <include filename="$(find frobo_description)/urdf/kinect_camera.urdf.xacro" />
-  <include filename="$(find frobo_description)/urdf/lidar.urdf.xacro" />
+  <xacro:include filename="$(find frobo_description)/urdf/base.urdf.xacro" />
+  <xacro:include filename="$(find frobo_description)/urdf/kinect_camera.urdf.xacro" />
+  <xacro:include filename="$(find frobo_description)/urdf/lidar.urdf.xacro" />
+  <!-- Import all Gazebo-customization elements, including Gazebo colors -->
+  <xacro:include filename="$(find frobo_description)/urdf/frobo.gazebo" />
+  <!-- Import Rviz colors -->
+  <xacro:include filename="$(find frobo_description)/urdf/materials.urdf.xacro" />
   <!-- Now we can start using the macros included above to define the actual Frobo -->
   <frobo_base name="base" color="Brown"/>

File: frobo_description/urdf/kinect_camera.urdf.xacro (robot description, xacro)
@@ -1,5 +1,5 @@
 <?xml version="1.0"?>
-<robot>
-  <macro name="kinect_camera" params="name parent *origin">
+<robot xmlns:xacro="http://www.ros.org/wiki/xacro">
+  <xacro:macro name="kinect_camera" params="name parent *origin">
     <joint name="${name}_frame_joint" type="fixed">
       <insert_block name="origin" />
@@ -65,4 +65,4 @@
     </joint>
     <link name="${name}_rgb_optical_frame"/>
-  </macro>
+  </xacro:macro>
 </robot>

File: frobo_description/urdf/lidar.urdf.xacro (robot description, xacro)
@@ -1,8 +1,8 @@
 <?xml version="1.0"?>
-<robot>
+<robot xmlns:xacro="http://www.ros.org/wiki/xacro">
   <!-- define a lidar -->
-  <macro name="lidar" params="name parent *origin">
+  <xacro:macro name="lidar" params="name parent *origin">
     <joint name="${name}_joint" type="fixed">
-      <insert_block name="origin" />
+      <xacro:insert_block name="origin" />
       <parent link="${parent}"/>
       <child link="${name}_link"/>
@@ -18,4 +18,4 @@
       </visual>
     </link>
-  </macro>
+  </xacro:macro>
 </robot>

Commit message: gazebo model improvements: added laser, camera and base_controller plugins

File: frobo_description/urdf/base.urdf.xacro (robot description, xacro)
@@ -124,8 +124,16 @@
       </visual>
       -->
+      <!-- split collision object of base in two, one below lidar, and one on top lidar
+      to keep lidar free for object detection (otherwise it would be blocked by collision object) -->
       <collision>
-        <origin xyz="0 0 ${(level3_clearance+base_collision_top_clearance)/2}" rpy="0 0 0" />
+      <origin xyz="0 0 ${level2_clearance/2}" rpy="0 0 0" />
         <geometry>
-          <cylinder radius="${base_collision_radius}" length="${level3_clearance+base_collision_top_clearance}"/>
+          <cylinder radius="${base_collision_radius}" length="${level2_clearance}"/>
+        </geometry>
+      </collision>
+      <collision>
+        <origin xyz="0 0 ${level3_clearance+base_collision_top_clearance/2}" rpy="0 0 0" />
+        <geometry>
+          <cylinder radius="${base_collision_radius}" length="${base_collision_top_clearance}"/>
         </geometry>
       </collision>

File: frobo_description/urdf/frobo.urdf (robot description, URDF)
Before this commit: robot frobo, 10 links, 9 joints
Links:
- removed link head_camera_frame
- removed link head_camera_ir_link
- removed link head_camera_ir_optical_frame
- removed link head_camera_rgb_link
- added link head_camera_depth_frame
- added link head_camera_depth_optical_frame
- added link head_camera_link; collision mesh filename=package://frobo_description/meshes/kinect_camera_simple.stl; visual mesh filename=package://frobo_description/meshes/kinect_camera_simple.dae
- added link head_camera_rgb_frame
- link base_link: geometry collision cylinder length=0.1 radius=0.2; collision cylinder length=0.24 radius=0.2
Joints:
- removed joint head_camera_frame_joint
- removed joint head_camera_ir_joint
- removed joint head_camera_ir_optical_frame_joint
- removed joint head_camera_rgb_optical_frame_joint
- added joint head_camera_depth_joint: type fixed, parent head_camera_link, child head_camera_depth_frame, origin xyz=0.0 -0.02 0.0 rpy=0 0 0
- added joint head_camera_depth_optical_joint: type fixed, parent head_camera_depth_frame, child head_camera_depth_optical_frame, origin xyz=0 0 0 rpy=-1.57079632679 0.0 -1.57079632679
- added joint head_camera_joint: type fixed, parent base_link, child head_camera_link, origin xyz=0 0 0.35 rpy=0 0 0
- added joint head_camera_rgb_optical_joint: type fixed, parent head_camera_rgb_frame, child head_camera_rgb_optical_frame, origin xyz=0 0 0 rpy=-1.57079632679 0.0 -1.57079632679
- joint head_camera_rgb_joint: child head_camera_rgb_link -> head_camera_rgb_frame; origin xyz=0 -0.03 0 rpy=0 0 0 -> xyz=0.0 -0.0125 0.0 rpy=0 0 0; parent head_camera_ir_link -> head_camera_link

File: frobo_description/urdf/frobo.urdf.xacro (robot description, xacro)
@@ -19,3 +19,5 @@
     <origin xyz="-0.02 0 0.285" rpy="0 0 0"/>
   </lidar>
+  <!-- extensions -->
+  <xacro:frobo_base_gazebo />
 </robot>

File: frobo_description/urdf/kinect_camera.urdf.xacro (robot description, xacro)
@@ -1,68 +1,55 @@
 <?xml version="1.0"?>
-<robot xmlns:xacro="http://www.ros.org/wiki/xacro">
-  <xacro:macro name="kinect_camera" params="name parent *origin">
-    <joint name="${name}_frame_joint" type="fixed">
-      <insert_block name="origin" />
-      <parent link="${parent}"/>
-      <child link="${name}_frame"/>
-    </joint>
-    <link name="${name}_frame">
-      <visual>
-        <origin xyz="-0.03 0 0.02" rpy="0 0 -1.57" />
-        <!--origin xyz="-0.03 -0.07 0" rpy="0 0 -1.57"-->
-        <geometry>
-          <mesh filename="package://frobo_description/meshes/kinect.stl" />
-        </geometry>
-        <material name="Black" />
-      </visual>
-      <collision>
-        <origin xyz="0 0 0" rpy="0 0 0" />
-        <geometry>
-          <box size="0.064 0.28 0.04"/>
-        </geometry>
-      </collision>
-    </link>
-    <!-- kinect ir sensor physical attachment -->
-    <joint name="${name}_ir_joint" type="fixed">
-      <origin xyz="0 0 0" rpy="0 0 0"/>
-      <parent link="${name}_frame"/>
-      <child link="${name}_ir_link"/>
-    </joint>
-    <link name="${name}_ir_link">
-      <visual>
-        <origin xyz="0.0 0.0 0" rpy="0 0 0"/>
-        <geometry>
-          <sphere radius="0.0005"/>
-        </geometry>
-      </visual>
-    </link>
-    <!-- kinect ir sensor frame -->
-    <joint name="${name}_ir_optical_frame_joint" type="fixed">
-      <origin xyz="0 0 0" rpy="-1.57 0.0 -1.57" />
-      <parent link="${name}_ir_link"/>
-      <child link="${name}_ir_optical_frame"/>
-    </joint>
-    <link name="${name}_ir_optical_frame"/>
-    <!-- kinect rgb sensor physical attachment -->
-    <joint name="${name}_rgb_joint" type="fixed">
-      <origin xyz="0 -0.03 0" rpy="0 0 0"/>
-      <parent link="${name}_ir_link"/>
-      <child link="${name}_rgb_link"/>
-    </joint>
-    <link name="${name}_rgb_link">
-      <visual>
-        <origin xyz="0.0 0.0 0" rpy="0 0 0"/>
-        <geometry>
-          <sphere radius="0.0005"/>
-        </geometry>
-      </visual>
-    </link>
-    <!-- kinect rgb sensor frame -->
-    <joint name="${name}_rgb_optical_frame_joint" type="fixed">
-      <origin xyz="0 0 0" rpy="-1.57 0.0 -1.57" />
-      <parent link="${name}_rgb_link"/>
-      <child link="${name}_rgb_optical_frame"/>
-    </joint>
-    <link name="${name}_rgb_optical_frame"/>
-  </xacro:macro>
+<robot xmlns:xacro="http://ros.org/wiki/xacro">
+    <xacro:property name="M_PI" value="3.1415926535897931" />
+    <xacro:macro name="kinect_camera_model" params="name parent *origin">
+      <joint name="${name}_joint" type="fixed">
+        <xacro:insert_block name="origin" />
+        <parent link="${parent}"/>
+        <child link="${name}_link"/>
+      </joint>
+      <link name="${name}_link">
+        <inertial_sphere mass="0.01" diameter="0.07" />
+        <visual>
+          <origin xyz="0 0 0" rpy="0 0 0" />
+          <geometry>
+            <mesh filename="package://frobo_description/meshes/kinect_camera_simple.dae"/>
+          </geometry>
+        </visual>
+        <collision>
+          <origin xyz="0 0 0" rpy="0 0 0" />
+          <geometry>
+            <mesh filename="package://frobo_description/meshes/kinect_camera_simple.stl"/>
+          </geometry>
+        </collision>
+      </link>
+      <joint name="${name}_depth_joint" type="fixed">
+        <origin xyz="0.0 -0.02 0.0" rpy="0 0 0" />
+        <parent link="${name}_link" />
+        <child link="${name}_depth_frame"/>
+      </joint>
+      <link name="${name}_depth_frame"/>
+      <joint name="${name}_depth_optical_joint" type="fixed">
+        <origin xyz="0 0 0" rpy="${-M_PI/2} 0.0 ${-M_PI/2}" />
+        <parent link="${name}_depth_frame" />
+        <child link="${name}_depth_optical_frame"/>
+      </joint>
+      <link name="${name}_depth_optical_frame"/>
+      <joint name="${name}_rgb_joint" type="fixed">
+        <origin xyz="0.0 -0.0125 0.0" rpy="0 0 0" />
+        <parent link="${name}_link" />
+        <child link="${name}_rgb_frame"/>
+      </joint>
+      <link name="${name}_rgb_frame"/>
+      <joint name="${name}_rgb_optical_joint" type="fixed">
+        <origin xyz="0 0 0" rpy="${-M_PI/2} 0.0 ${-M_PI/2}" />
+        <parent link="${name}_rgb_frame" />
+        <child link="${name}_rgb_optical_frame"/>
+      </joint>
+      <link name="${name}_rgb_optical_frame"/>
+    </xacro:macro>
+    <xacro:macro name="kinect_camera" params="name parent *origin">
+      <xacro:kinect_camera_model name="${name}" parent="${parent}">
+        <xacro:insert_block name="origin" />
+      </xacro:kinect_camera_model>
+    </xacro:macro>
 </robot>

Commit message: frobo_description: introduce base_footprint link

File: frobo_description/urdf/base.urdf.xacro (robot description, xacro)
@@ -68,6 +68,33 @@
   </xacro:macro>
   <!-- The xacro macro frobo_base contains: base and wheels -->
-  <xacro:macro name="frobo_base" params="name color">
-    <link name="${name}_link">
+  <xacro:macro name="frobo_base" params="color">
+    <link name="base_footprint">
+      <visual>
+        <origin xyz="0 0 0" rpy="0 0 0"/>
+        <geometry>
+          <box size="0.001 0.001 0.001"/>
+        </geometry>
+        <material name="Black" />
+      </visual>
+      <collision>
+        <origin xyz="0 0 ${ground_clearance}" rpy="0 0 0"/>
+        <geometry>
+         <box size="0.001 0.001 0.001"/>
+        </geometry>
+      </collision>
+    </link>
+    <!--
+        base_footprint mapping was introduced as robot-pose-ekf requires it.
+        strictly spoken, base_link should be attached to the base,
+	and base_footprint is a projection of base_link on the ground.
+        Here base_link and base_footprint are simply mapped on the same point, on the ground.
+        See also https://github.com/ros-planning/navigation/issues/15
+    -->
+    <joint name="base_joint" type="fixed">
+      <origin xyz="0 0 0" rpy="0 0 0" />
+      <parent link="base_footprint"/>
+      <child link="base_link" />
+    </joint>
+    <link name="base_link">
       <visual>
         <origin xyz="0 0 ${ground_clearance}" rpy="0 0 0" />
@@ -127,5 +154,5 @@
       to keep lidar free for object detection (otherwise it would be blocked by collision object) -->
       <collision>
-      <origin xyz="0 0 ${level2_clearance/2}" rpy="0 0 0" />
+        <origin xyz="0 0 ${level2_clearance/2}" rpy="0 0 0" />
         <geometry>
           <cylinder radius="${base_collision_radius}" length="${level2_clearance}"/>
@@ -151,7 +178,7 @@
     <frobo_wheel parent="${name}" suffix="r" reflect="-1" color="Orange"/>-->
     <!-- sonars -->
-    <frobo_sonar parent="${name}" offset_x="0.115" offset_y="-0.055" angle="-${sonar_angle}" suffix="fr" color="Blue"/>
-    <frobo_sonar parent="${name}" offset_x="0.125" offset_y="0" angle="0" suffix="fc" color="Blue"/>
-    <frobo_sonar parent="${name}" offset_x="0.115" offset_y="0.055" angle="${sonar_angle}" suffix="fl" color="Blue"/>
+    <frobo_sonar parent="base" offset_x="0.115" offset_y="-0.055" angle="-${sonar_angle}" suffix="fr" color="Blue"/>
+    <frobo_sonar parent="base" offset_x="0.125" offset_y="0" angle="0" suffix="fc" color="Blue"/>
+    <frobo_sonar parent="base" offset_x="0.115" offset_y="0.055" angle="${sonar_angle}" suffix="fl" color="Blue"/>
   </xacro:macro>
 </robot>

File: frobo_description/urdf/frobo.urdf.xacro (robot description, xacro)
@@ -10,5 +10,5 @@
   <xacro:include filename="$(find frobo_description)/urdf/materials.urdf.xacro" />
   <!-- Now we can start using the macros included above to define the actual Frobo -->
-  <frobo_base name="base" color="Brown"/>
+  <frobo_base color="Brown"/>
   <!-- Camera -->
   <kinect_camera name="head_camera" parent="base_link">
