Commit message: frobo_description: adding imu

File: frobo_description/urdf/base.urdf.xacro (robot description, xacro)
@@ -1,5 +1,14 @@
 <?xml version="1.0"?>
 <robot xmlns:xacro="http://www.ros.org/wiki/xacro">
-  <xacro:property name="ground_clearance" value="0.0740" />
+<!-- Grey wheels -->
+  <xacro:property name="ground_clearance" value="0.0495" />
+  <xacro:property name="level1_clearance" value="0.16" />
+  <xacro:property name="level2_clearance" value="0.215" />
+  <xacro:property name="level3_clearance" value="0.275" />
+  <xacro:property name="wheel_offset_y" value="0.116" />
+  <xacro:property name="wheel_length" value="0.02032" />
+  <xacro:property name="wheel_radius" value="0.0375" />
+<!-- Orange wheels -->
+<!--  <xacro:property name="ground_clearance" value="0.0740" />
   <xacro:property name="level1_clearance" value="0.18" />
   <xacro:property name="level2_clearance" value="0.24" />
@@ -7,5 +16,5 @@
   <xacro:property name="wheel_offset_y" value="0.116" />
   <xacro:property name="wheel_length" value="0.02032" />
-  <xacro:property name="wheel_radius" value="0.06191" />
+  <xacro:property name="wheel_radius" value="0.06191" /> -->
   <xacro:property name="swivel_length" value="0.019" />
   <xacro:property name="swivel_radius" value="0.025" />
@@ -132,5 +141,5 @@
           <cylinder radius="${wheel_radius}" length="${wheel_length}"/>
         </geometry>
-        <material name="Orange" />
+        <material name="Grey" />
       </visual>
       <visual>
@@ -139,5 +148,5 @@
           <cylinder radius="${wheel_radius}" length="${wheel_length}"/>
         </geometry>
-        <material name="Orange" />
+        <material name="Grey" />
       </visual>
       <!-- fixed swivel, without tf transform, just for visualization -->

File: frobo_description/urdf/frobo.urdf.xacro (robot description, xacro)
@@ -5,4 +5,5 @@
   <xacro:include filename="$(find frobo_description)/urdf/kinect_camera.urdf.xacro" />
   <xacro:include filename="$(find frobo_description)/urdf/lidar.urdf.xacro" />
+  <xacro:include filename="$(find frobo_description)/urdf/imu.urdf.xacro" />
   <!-- Import all Gazebo-customization elements, including Gazebo colors -->
   <xacro:include filename="$(find frobo_description)/urdf/frobo.gazebo" />
@@ -13,10 +14,14 @@
   <!-- Camera -->
   <kinect_camera name="head_camera" parent="base_link">
-    <origin xyz="0 0 0.35" rpy="0 0 0"/>
+    <origin xyz="0 0 0.32" rpy="0 0 0"/>
   </kinect_camera>
   <!-- Lidar -->
   <lidar name="lidar" parent="base_link">
-    <origin xyz="-0.02 0 0.285" rpy="0 0 0"/>
+    <origin xyz="-0.02 0 0.26" rpy="0 0 0"/>
   </lidar>
+  <!-- IMU -->
+  <imu name="base_imu" parent="base_link">
+    <origin xyz="0 0 0.28" rpy="0 0 0"/>
+  </imu>
   <!-- extensions -->
   <xacro:frobo_base_gazebo />

Commit message: frobo_description: updating urdf in line with latest build

File: frobo_description/urdf/base.urdf.xacro (robot description, xacro)
@@ -2,8 +2,8 @@
 <robot xmlns:xacro="http://www.ros.org/wiki/xacro">
 <!-- Grey wheels -->
-  <xacro:property name="ground_clearance" value="0.0495" />
-  <xacro:property name="level1_clearance" value="0.16" />
-  <xacro:property name="level2_clearance" value="0.215" />
-  <xacro:property name="level3_clearance" value="0.275" />
+  <xacro:property name="ground_clearance" value="0.053" />
+  <xacro:property name="level1_clearance" value="0.1175" />
+  <xacro:property name="level2_clearance" value="0.180" />
+  <xacro:property name="level3_clearance" value="0.282" />
   <xacro:property name="wheel_offset_y" value="0.116" />
   <xacro:property name="wheel_length" value="0.02032" />
@@ -187,7 +187,7 @@
     <frobo_wheel parent="${name}" suffix="r" reflect="-1" color="Orange"/>-->
     <!-- sonars -->
-    <frobo_sonar parent="base" offset_x="0.115" offset_y="-0.055" angle="-${sonar_angle}" suffix="fr" color="Blue"/>
+    <!--<frobo_sonar parent="base" offset_x="0.115" offset_y="-0.055" angle="-${sonar_angle}" suffix="fr" color="Blue"/>
     <frobo_sonar parent="base" offset_x="0.125" offset_y="0" angle="0" suffix="fc" color="Blue"/>
-    <frobo_sonar parent="base" offset_x="0.115" offset_y="0.055" angle="${sonar_angle}" suffix="fl" color="Blue"/>
+    <frobo_sonar parent="base" offset_x="0.115" offset_y="0.055" angle="${sonar_angle}" suffix="fl" color="Blue"/>-->
   </xacro:macro>
 </robot>

File: frobo_description/urdf/frobo.urdf.xacro (robot description, xacro)
@@ -14,14 +14,14 @@
   <!-- Camera -->
   <kinect_camera name="head_camera" parent="base_link">
-    <origin xyz="0 0 0.32" rpy="0 0 0"/>
+    <origin xyz="0 0.002 0.345" rpy="0 0 0"/>
   </kinect_camera>
   <!-- Lidar -->
   <lidar name="lidar" parent="base_link">
-    <origin xyz="-0.02 0 0.26" rpy="0 0 0"/>
+    <origin xyz="-0.02 0 0.165" rpy="0 0 0"/>
   </lidar>
   <!-- IMU -->
-  <imu name="base_imu" parent="base_link">
+ <!-- <imu name="base_imu" parent="base_link">
     <origin xyz="0 0 0.28" rpy="0 0 0"/>
-  </imu>
+  </imu>-->
   <!-- extensions -->
   <xacro:frobo_base_gazebo />

Commit message: frobo_description: updating with new lidar position

File: frobo_description/urdf/base.urdf.xacro (robot description, xacro)
@@ -4,5 +4,5 @@
   <xacro:property name="ground_clearance" value="0.053" />
   <xacro:property name="level1_clearance" value="0.1175" />
-  <xacro:property name="level2_clearance" value="0.180" />
+  <xacro:property name="level2_clearance" value="0.1875" />
   <xacro:property name="level3_clearance" value="0.282" />
   <xacro:property name="wheel_offset_y" value="0.116" />

File: frobo_description/urdf/frobo.urdf.xacro (robot description, xacro)
@@ -18,5 +18,5 @@
   <!-- Lidar -->
   <lidar name="lidar" parent="base_link">
-    <origin xyz="-0.02 0 0.165" rpy="0 0 0"/>
+    <origin xyz="-0.051 0 0.1725" rpy="0 0 0"/>
   </lidar>
   <!-- IMU -->
