Commit message: frobo_description: adding swivel

File: frobo_description/urdf/base.urdf.xacro (robot description, xacro)
@@ -60,5 +60,5 @@
       </collision>
       <inertial>
-        <origin xyz="0 0 ${wheel_radius}" rpy="0 0 0"/>
+        <origin xyz="0 0 0" rpy="0 0 0"/>
         <mass value="0.2"/>
         <inertia
@@ -123,4 +123,61 @@
 	    </geometry>
       </visual>
+  </xacro:macro>
+  <!-- define swivel -->
+  <xacro:macro name="frobo_swivel" params="parent color offset_x offset_z">
+    <joint name="base_to_rear_wheel" type="fixed">
+      <parent link="${parent}_link"/>
+      <child link="swivel_bottom"/>
+      <origin xyz="${offset_x} 0 ${-0.01615+offset_z}" rpy="0 0 0"/>
+    </joint>
+    <link name="swivel_bottom">
+       <visual>
+        <origin xyz="0 0 0" rpy="0 0 0" />
+        <geometry>
+          <box size="0.005 0.005 0.0323"/>
+        </geometry>
+        <material name="Grey" />
+      </visual>
+      <collision>
+        <origin xyz="0 0 0" rpy="0 0 0" />
+        <geometry>
+           <box size="0.005 0.005 0.0323"/>
+        </geometry>
+      </collision>
+      <inertial>
+       <mass value="0.1" />
+       <inertia ixx="0.001" ixy="0.0" ixz="0.0"
+                   iyy="0.001" iyz="0.0"
+                   izz="0.001" />
+      </inertial>
+    </link>
+    <joint name="swivel_joint" type="fixed">
+     <parent link="swivel_bottom"/>
+     <child link="${parent}_swivel_link" />
+     <origin xyz="0 0 -0.01615" rpy="${PI/2} 0 0" />
+    </joint>
+    <link name="${parent}_swivel_link">
+      <visual>
+        <geometry>
+          <cylinder radius="0.016" length="0.015"/>
+        </geometry>
+        <origin xyz="0 0 0" rpy="0 0 0"/>
+        <material name="${color}"/>
+      </visual>
+      <collision>
+        <geometry>
+          <cylinder radius="0.016" length="0.015"/>
+        </geometry>
+        <origin xyz="0 0 0" rpy="0 0 0"/>
+      </collision>
+      <inertial>
+          <origin xyz="0 0 0" rpy="0 0 0"/>
+          <mass value="0.01"/>
+          <inertia
+            ixx="0.01" ixy="0.0" ixz="0.0"
+            iyy="0.01" iyz="0.0"
+            izz="0.01"/>
+      </inertial>
+    </link>
   </xacro:macro>
   <!-- define base -->
@@ -169,4 +226,5 @@
 -->
       <!-- fixed swivel, without tf transform, just for visualization -->
+<!--
       <visual>
         <origin xyz="-${wheel_offset_y} 0 -${swivel_radius+base_thickness/2}" rpy="${PI/2} 0 0" />
@@ -175,4 +233,5 @@
         </geometry>
       </visual>
+-->
       <!-- basic collision protection, make sure to keep camera and lidar free for object detection
       (otherwise it would be blocked by collision object) -->
@@ -184,5 +243,5 @@
       </collision>
       <inertial>
-        <origin xyz="0 0 ${base_radius}" rpy="0 0 0"/>
+        <origin xyz="0 0 0" rpy="0 0 0"/>
         <mass value="5"/>
         <inertia
@@ -201,4 +260,6 @@
     <frobo_wheel parent="base" suffix="l" reflect="1" color="${wheel_color}"/>
     <frobo_wheel parent="base" suffix="r" reflect="-1" color="${wheel_color}"/>
+    <!-- rotating swivel -->
+    <frobo_swivel parent="base" color="Black" offset_x="-0.13" offset_z="-${base_thickness/2}"/>
     <!-- sonars -->
     <frobo_sonar parent="base" offset_x="0.115" offset_y="-0.055" angle="-${sonar_angle}" suffix="fr" color="Blue"/>

Commit message: frobo_description: updating measurements

File: frobo_description/urdf/base.urdf.xacro (robot description, xacro)
@@ -28,5 +28,5 @@
   <xacro:property name="level2_clearance" value="0.065" />
   <!-- level3_clearance: distance between bottom level 2 plate and top level 3 plate (NOT centers) -->
-  <xacro:property name="level3_clearance" value="0.086" />
+  <xacro:property name="level3_clearance" value="0.09" />
   <xacro:property name="base_mesh_scale" value="1" />
   <xacro:property name="swivel_length" value="0.019" />
@@ -39,4 +39,5 @@
     <joint name="${parent}_${suffix}_wheel_joint" type="continuous">
       <axis xyz="0 0 1" />
+      <anchor xyz="0 0 0" />
       <limit effort="100" velocity="100"/>
       <safety_controller k_velocity="10" />
@@ -130,4 +131,5 @@
       <child link="swivel_bottom"/>
       <origin xyz="${offset_x} 0 ${-0.01615+offset_z}" rpy="0 0 0"/>
+      <anchor xyz="0 0 1" />
     </joint>
     <link name="swivel_bottom">

File: frobo_description/urdf/lidar.urdf.xacro (robot description, xacro)
@@ -1,10 +1,10 @@
 <?xml version="1.0"?>
 <robot xmlns:xacro="http://www.ros.org/wiki/xacro">
-  <xacro:property name="lidar_box_size_x" value="0.124" />
+  <xacro:property name="lidar_box_size_x" value="0.126" />
   <xacro:property name="lidar_box_size_y" value="0.105" />
   <xacro:property name="lidar_box_size_z" value="0.048" />
-  <xacro:property name="lidar_radius" value="0.038" />
+  <xacro:property name="lidar_radius" value="0.039" />
   <!-- offset relative to box - how much it sticks out on top -->
-  <xacro:property name="lidar_offset_z" value="0.01" />
+  <xacro:property name="lidar_offset_z" value="0.013" />
   <!-- define a lidar -->
   <xacro:macro name="lidar" params="name parent *origin">
